Commit message: implement lane node skeleton

File: src/sedan_description/urdf/sedan.urdf.xacro (robot description, xacro)
@@ -51,5 +51,5 @@
         <parent link="base_link" />
         <child link="chassis" />
-        <origin xyz="0 0 ${wheel_radius + ch_h/2}" rpy="0 0 0" />
+        <origin xyz="0 0 ${wheel_radius}" rpy="0 0 0" />
     </joint>
     <link name="chassis">
@@ -97,5 +97,5 @@
             <parent link="chassis" />
             <child link="${prefix}_wheel_steering_link" />
-            <origin xyz="${x_off} ${y_off} ${-ch_h/2}" rpy="0 0 0" />
+            <origin xyz="${x_off} ${y_off} 0" rpy="0 0 0" />
             <axis xyz="0 0 1" />
             <!-- velocity 2.5 (power steering at low speed) + light damping: the
@@ -125,9 +125,9 @@
     </xacro:macro>
     <!-- ===================== WHEEL MACRO ===================== -->
-    <xacro:macro name="wheel" params="name parent x_off y_off">
+    <xacro:macro name="wheel" params="name parent x_off y_off z_off">
         <joint name="${name}_joint" type="continuous">
             <parent link="${parent}" />
             <child link="${name}" />
-            <origin xyz="${x_off} ${y_off} 0" rpy="0 0 0" />
+            <origin xyz="${x_off} ${y_off} ${z_off}" rpy="0 0 0" />
             <axis xyz="0 1 0" />
         </joint>
@@ -155,16 +155,16 @@
     <xacro:steering_link prefix="front_right" x_off="${wheelbase/2}" y_off="${-track_width/2}" />
     <xacro:wheel name="front_left_wheel"
-        parent="front_left_wheel_steering_link" x_off="0" y_off="0" />
+        parent="front_left_wheel_steering_link" x_off="0" y_off="0" z_off="0" />
     <xacro:wheel name="front_right_wheel"
-        parent="front_right_wheel_steering_link" x_off="0" y_off="0" />
+        parent="front_right_wheel_steering_link" x_off="0" y_off="0" z_off="0" />
     <xacro:wheel name="rear_left_wheel"
-        parent="chassis" x_off="${-wheelbase/2}" y_off="${track_width/2}" />
+        parent="chassis" x_off="${-wheelbase/2}" y_off="${track_width/2}" z_off="0" />
     <xacro:wheel name="rear_right_wheel"
-        parent="chassis" x_off="${-wheelbase/2}" y_off="${-track_width/2}" />
+        parent="chassis" x_off="${-wheelbase/2}" y_off="${-track_width/2}" z_off="0" />
     <!-- ===================== FRONT CAMERA ===================== -->
     <joint name="front_camera_joint" type="fixed">
-        <parent link="base_link" />
+        <parent link="chassis" />
         <child link="front_camera_link" />
-        <origin xyz="${cam_x} 0 ${cam_z}" rpy="0 ${cam_pitch} 0" />
+        <origin xyz="${cam_x} 0 ${cam_z - wheel_radius}" rpy="0 ${cam_pitch} 0" />
     </joint>
     <link name="front_camera_link">
@@ -217,7 +217,7 @@
     <!-- ===================== IMU ===================== -->
     <joint name="imu_joint" type="fixed">
-        <parent link="base_link" />
+        <parent link="chassis" />
         <child link="imu_link" />
-        <origin xyz="0 0 ${wheel_radius + ch_h/2}" rpy="0 0 0" />
+        <origin xyz="0 0 0" rpy="0 0 0" />
     </joint>
     <link name="imu_link">

Commit message: commit before mpc update for steering slew rate

File: src/sedan_description/urdf/sedan.urdf.xacro (robot description, xacro)
@@ -99,10 +99,30 @@
             <origin xyz="${x_off} ${y_off} 0" rpy="0 0 0" />
             <axis xyz="0 0 1" />
-            <!-- velocity 2.5 (power steering at low speed) + light damping: the
-           1.0 rad/s + damping 5 actuator lagged the MPC into a bang-bang
-           steering limit cycle (2026-07-11 steer probe). The MPC node also
-           slew-limits its command to steer_slew_rps to match. -->
-            <limit lower="-0.55" upper="0.55" effort="400.0" velocity="2.5" />
-            <dynamics damping="2.0" />
+            <!-- damping=2.0, confirmed by a 0/0.5/2.0 same-day A/B/C sweep
+           (2026-09-04) to have NO measurable effect on the fast e_head/steer
+           chatter seen mid-course - that chatter tracks a location on the
+           path, not this value. Left at 2.0, the pre-2026-09-04 default.
+           velocity 2.5 -> 4.0 (2026-09-04): the QP's internal vehicle model
+           (mpc_solver/vehicle_model.cpp) has NO steering-rate state - delta
+           is a free variable at every 0.12s horizon step, achievable
+           instantly as far as the optimizer knows. The plant's real cap was
+           2.5 rad/s, i.e. >=0.48s for a full +/-0.6 rad swing (4 horizon
+           steps) - a genuine plan-vs-plant rate gap, same bug class as the
+           max_steer_rad-vs-steering_limit MAGNITUDE mismatch fixed earlier
+           this session, just for RATE instead. Raised to 4.0, above the MPC
+           node's own steer_slew_rps (3.0 rad/s, mpc_params.yaml) output
+           limiter, so that explicit, tunable software limit - not this
+           buried joint value - is now the sole binding rate constraint the
+           plant approximately respects. The QP still doesn't reason about
+           steer_slew_rps internally; this only narrows the gap, it doesn't
+           close it (that needs a rate-limited delta state in the model). -->
+            <!-- kept 0.05 rad above <steering_limit> in the AckermannSteering
+           plugin below, same margin style: this joint limit is the hard
+           mechanical stop, the plugin's steering_limit is what it actually
+           commands, so the plugin should always bind first. Raising one
+           without the other reproduces the max_steer_rad-vs-steering_limit
+           mismatch bug (2026-09-04 turn-settling diagnosis) one level down. -->
+            <limit lower="-0.70" upper="0.70" effort="400.0" velocity="4.0" />
+            <dynamics damping="0.0" />
         </joint>
         <link name="${prefix}_wheel_steering_link">
@@ -162,4 +182,50 @@
     <xacro:wheel name="rear_right_wheel"
         parent="chassis" x_off="${-wheelbase/2}" y_off="${-track_width/2}" z_off="0" />
+    <!-- ===================== WHEEL FRICTION (slip1/slip2) ===================== -->
+    <!-- ODE surface friction via the <gazebo reference><collision><surface> path:
+       sdformat's URDF converter has two mechanisms for <gazebo reference> collision
+       props - a narrow flat whitelist (mu1/mu2/kp/kd/maxVel/minDepth, direct
+       children) and a "blob" path where a nested <collision> child is inserted
+       into the output SDF verbatim. slip1/slip2 aren't in the whitelist, so this
+       has to go through the blob path (nest under <collision>, not flat).
+       mu/mu2 = 1.0 keeps the Coulomb traction ceiling unchanged; slip1/slip2 add
+       continuous, tunable compliance so a wheel can slip under load instead of an
+       all-or-nothing traction cliff (lower risk on this rigid 300 kg body with no
+       tire model - see the mass-choice note up top). This is what lets the front
+       (steered) wheels slip laterally in a tight turn, which breaks the
+       AckermannSteering odometry's no-slip bicycle-model assumption for yaw
+       (phi -> yaw) while the IMU gyro keeps measuring the true chassis rotation -
+       i.e. this is the mechanism for making /odom_ekf beat raw /odom under load.
+       Values are a first guess, not derived - tune empirically against the
+       odom_truth_spawn vs /odom vs /odom_ekf divergence in a tight turn
+       (generate_course_world.py's turn radius flag).
+       Default slip is 0.0 (disabled) as of the 2026-09-04 turn-settling
+       diagnosis: with slip at 0.02 the MPC's no-slip bicycle model
+       (mpc_solver's integrate_kinematic) was seeing ~1.5x less cornering
+       authority than commanded, on top of a since-fixed max_steer_rad/
+       steering_limit mismatch. Re-enable (pass slip="0.02" at the call
+       sites below) once ready to resume the /odom_ekf-beats-/odom
+       experiment, ideally with the truth-vs-EKF yaw rate check run first
+       to confirm how much of that deficit is real slip vs. estimator lag. -->
+    <xacro:macro name="wheel_friction" params="link slip:=0.0">
+        <gazebo reference="${link}">
+            <collision>
+                <surface>
+                    <friction>
+                        <ode>
+                            <mu>1.0</mu>
+                            <mu2>1.0</mu2>
+                            <slip1>${slip}</slip1>
+                            <slip2>${slip}</slip2>
+                        </ode>
+                    </friction>
+                </surface>
+            </collision>
+        </gazebo>
+    </xacro:macro>
+    <xacro:wheel_friction link="front_left_wheel" />
+    <xacro:wheel_friction link="front_right_wheel" />
+    <xacro:wheel_friction link="rear_left_wheel" />
+    <xacro:wheel_friction link="rear_right_wheel" />
     <!-- ===================== FRONT CAMERA ===================== -->
     <joint name="front_camera_joint" type="fixed">
@@ -200,5 +266,13 @@
             <right_steering_joint>front_right_wheel_steering_joint</right_steering_joint>
             <kingpin_width>${track_width}</kingpin_width>
-            <steering_limit>0.50</steering_limit>
+            <!-- raised from 0.50 (2026-09-04): at 0.50 rad / wheelbase 2.7 m
+           the tightest achievable turn is ~4.9 m radius, too wide for
+           urban_tight's ~3.5 m-radius bends. 0.65 rad -> ~2.7/tan(0.65) =
+           3.55 m. Keep mpc_params.yaml's max_steer_rad a safety margin BELOW
+           this value (currently 0.05 rad, matching the joint <limit> margin
+           above) - the QP must never plan for more angle than the plant can
+           deliver, that mismatch was the root cause of the 2026-09-04
+           turn-settling bug. -->
+            <steering_limit>0.65</steering_limit>
             <wheel_base>${wheelbase}</wheel_base>
             <wheel_separation>${track_width}</wheel_separation>

Commit message: mpc tuning

File: src/sedan_description/urdf/sedan.urdf.xacro (robot description, xacro)
@@ -123,5 +123,5 @@
            without the other reproduces the max_steer_rad-vs-steering_limit
            mismatch bug (2026-09-04 turn-settling diagnosis) one level down. -->
-            <limit lower="-0.70" upper="0.70" effort="400.0" velocity="4.0" />
+            <limit lower="-0.80" upper="0.80" effort="400.0" velocity="4.0" />
             <dynamics damping="0.0" />
         </joint>

Commit message: reduce camera blind zone near the car

File: src/sedan_description/urdf/sedan.urdf.xacro (robot description, xacro)
@@ -24,6 +24,13 @@
     <xacro:property name="steer_mass" value="5.0" />
     <xacro:property name="wheel_mass" value="15.0" />
-    <!-- camera mount (day-03 memo: 1.4 m height buys ~25-35 m lane visibility) -->
-    <xacro:property name="cam_x" value="1.9" />
+    <!-- camera mount (day-03 memo: 1.4 m height buys ~25-35 m lane visibility).
+       cam_x 1.9->1.2 (2026-09-05): 1.9m put the mount near the front bumper;
+       1.2m is closer to a realistic windshield-area dashcam position for
+       this wheelbase, and directly shrinks the near-field blind zone (the
+       closest visible ground row, ~2.2m from the camera at cam_z=1.4/
+       pitch=0.06/424-wide-image geometry - see expected_ground_distance in
+       lane_node.cpp) by the same 0.7m, since it's a pure translation with
+       no effect on the pitch-driven near/far FOV tradeoff. -->
+    <xacro:property name="cam_x" value="1.2" />
     <xacro:property name="cam_z" value="1.4" />
     <xacro:property name="cam_pitch" value="0.06" />
@@ -389,9 +396,21 @@
                          can't sustain 10 Hz RGBD at 640x360 (stalled to ~3-4 Hz
                          with 1.6 s gaps); 320x180 was too coarse and starved
-                         the far paint blobs. 16:9 kept, so the derived pinhole
-                         geometry is unchanged (fx/fy just scale). If the far
-                         field still matters, line_area_min_px scales with it. -->
+                         the far paint blobs.
+                         height 240->300 (2026-09-05): width/horizontal_fov
+                         unchanged, so horizontal detail and far-field lateral
+                         resolution are untouched, but pinhole_from_config
+                         (ground_cal.hpp) sets fy=fx from width/hfov alone, so
+                         a taller image is a wider VERTICAL fov at the same
+                         fx - the near AND far ground-visibility limits both
+                         extend (see expected_ground_distance), instead of
+                         trading one for the other via cam_pitch alone. 424x300
+                         is ~25% more pixels than 424x240 (vs 640x360's 2.3x) -
+                         cheaper on the WSL software renderer than the earlier
+                         full-width bump that broke framerate. line_area_min_px
+                         (lane_node.cpp) scales with total pixel area, so it
+                         needs revisiting if this is kept (currently sized for
+                         424x240). -->
                     <width>424</width>
-                    <height>240</height>
+                    <height>300</height>
                     <format>R8G8B8</format>
                 </image>

Commit message: Add project README and RViz/Gazebo snapshots; narrow camera FOV, reduce hood occlusion, reintroduce small wheel slip
- README.md: project overview, attribution to kfan12/vlm_robot_public,
  stack breakdown, screenshots, quick-start launch commands.
- docs/snapshots/: gazebo.png and rviz.png illustrations for the README.
- .gitignore: track docs/snapshots while keeping av_daily_plans/teaching ignored.
- sedan.urdf.xacro / lane_node.cpp: camera width/height settled back to
  424x300 with horizontal_fov widened to 1.9 for near-field ground
  coverage instead of extra pixels; cam_x moved to 2.2 to clear hood
  self-occlusion; wheel_friction slip1/slip2 reintroduced at a small 0.01
  now that the steering-limit, steer-rate, and curvature-margin fixes
  are in place.

File: src/sedan_description/urdf/sedan.urdf.xacro (robot description, xacro)
@@ -25,12 +25,18 @@
     <xacro:property name="wheel_mass" value="15.0" />
     <!-- camera mount (day-03 memo: 1.4 m height buys ~25-35 m lane visibility).
-       cam_x 1.9->1.2 (2026-09-05): 1.9m put the mount near the front bumper;
-       1.2m is closer to a realistic windshield-area dashcam position for
-       this wheelbase, and directly shrinks the near-field blind zone (the
-       closest visible ground row, ~2.2m from the camera at cam_z=1.4/
-       pitch=0.06/424-wide-image geometry - see expected_ground_distance in
-       lane_node.cpp) by the same 0.7m, since it's a pure translation with
-       no effect on the pitch-driven near/far FOV tradeoff. -->
-    <xacro:property name="cam_x" value="1.2" />
+       cam_x 1.9->1.2->2.2 (2026-09-05): 1.2m shrank the near-field blind
+       zone (good) but put the camera far enough BEHIND the chassis's own
+       front edge (chassis spans +/-2.25m around base_link) that the car's
+       own hood intruded into the bottom of the frame once the vertical FOV
+       was also widened (height 240->300) - confirmed visually in
+       /lane/debug_image. At the ORIGINAL 1.9m the hood was never visible
+       (even before the height change), so 2.2m - close to the chassis's
+       own front edge - is chosen for real margin against hood self-
+       occlusion at the wider vertical FOV, at the cost of reopening part of
+       the near-field blind-zone gain (net still forward of the original
+       1.9m). If the hood still shows up at this value, cam_z (height) is
+       the other lever - it looks over the hood at a steeper angle instead
+       of moving past it horizontally. -->
+    <xacro:property name="cam_x" value="2.2" />
     <xacro:property name="cam_z" value="1.4" />
     <xacro:property name="cam_pitch" value="0.06" />
@@ -207,13 +213,18 @@
        odom_truth_spawn vs /odom vs /odom_ekf divergence in a tight turn
        (generate_course_world.py's turn radius flag).
-       Default slip is 0.0 (disabled) as of the 2026-09-04 turn-settling
+       Default slip was 0.0 (disabled) from the 2026-09-04 turn-settling
        diagnosis: with slip at 0.02 the MPC's no-slip bicycle model
        (mpc_solver's integrate_kinematic) was seeing ~1.5x less cornering
        authority than commanded, on top of a since-fixed max_steer_rad/
-       steering_limit mismatch. Re-enable (pass slip="0.02" at the call
-       sites below) once ready to resume the /odom_ekf-beats-/odom
-       experiment, ideally with the truth-vs-EKF yaw rate check run first
-       to confirm how much of that deficit is real slip vs. estimator lag. -->
-    <xacro:macro name="wheel_friction" params="link slip:=0.0">
+       steering_limit mismatch.
+       Re-enabled at a small 0.01 (2026-09-05, half the old 0.02) now that
+       the steering_limit mismatch, steer-rate hard constraint, and
+       curvature-relative steering margin are all in place - a smaller
+       first step to resume the /odom_ekf-beats-/odom experiment without
+       repeating the same cornering-authority deficit. Raise toward 0.02
+       once this is confirmed not to reopen it; ideally with the
+       truth-vs-EKF yaw rate check run first to isolate real slip from
+       estimator lag. -->
+    <xacro:macro name="wheel_friction" params="link slip:=0.01">
         <gazebo reference="${link}">
             <collision>
@@ -391,5 +402,20 @@
             <update_rate>10</update_rate>
             <camera>
-                <horizontal_fov>1.6</horizontal_fov>
+                <!-- horizontal_fov 1.6->1.9 (2026-09-05): pinhole_from_config
+                     (ground_cal.hpp) derives fx=fy=(w/2)/tan(hfov/2), and
+                     expected_ground_distance's near-ground-row term
+                     ((v-cy)/fy) is the dominant factor in how close the
+                     visible ground gets (far more leverage than cam_pitch -
+                     a 0.06->0.30 rad pitch sweep only moved the near limit
+                     ~8%, this hfov change alone moves it ~30%). Raising hfov
+                     lowers fx=fy at the same width, which widens the
+                     VERTICAL fov too (same mechanism as the width/height
+                     notes below) and pulls the near-field ground limit
+                     forward. Left cam_pitch untouched deliberately: tilting
+                     down further is the OTHER way to gain near coverage but
+                     it eats into the cam_x=2.2 hood-clearance margin;
+                     widening hfov does not. 1.9 rad = ~109 deg total, wide
+                     but plausible for a low-mounted ADAS-style lane camera. -->
+                <horizontal_fov>1.9</horizontal_fov>
                 <image>
                     <!-- 424x240 (was 640x360): the WSL software-GL renderer
@@ -397,18 +423,17 @@
                          with 1.6 s gaps); 320x180 was too coarse and starved
                          the far paint blobs.
-                         height 240->300 (2026-09-05): width/horizontal_fov
-                         unchanged, so horizontal detail and far-field lateral
-                         resolution are untouched, but pinhole_from_config
-                         (ground_cal.hpp) sets fy=fx from width/hfov alone, so
-                         a taller image is a wider VERTICAL fov at the same
-                         fx - the near AND far ground-visibility limits both
-                         extend (see expected_ground_distance), instead of
-                         trading one for the other via cam_pitch alone. 424x300
-                         is ~25% more pixels than 424x240 (vs 640x360's 2.3x) -
-                         cheaper on the WSL software renderer than the earlier
-                         full-width bump that broke framerate. line_area_min_px
-                         (lane_node.cpp) scales with total pixel area, so it
-                         needs revisiting if this is kept (currently sized for
-                         424x240). -->
+                         width/height churned 424x240 -> 500x400 -> 400x400
+                         (2026-09-05) chasing near-field ground coverage by
+                         widening the vertical FOV (pinhole_from_config sets
+                         fy=fx from width/hfov, so a taller image at the same
+                         fx is a wider vertical FOV - see expected_ground_
+                         distance); settled back to 424x300 (101376 px,
+                         ~1.0x the original baseline, well clear of 640x360's
+                         2.26x that broke framerate) once horizontal_fov
+                         (1.6->1.9, see above) took over as the near-field
+                         lever instead - it gets the same fy reduction
+                         without spending extra pixels on it.
+                         line_area_min_px (lane_node.cpp) scales with total
+                         pixel area - updated for 424x300 alongside this. -->
                     <width>424</width>
                     <height>300</height>

Commit message: adjust img size

File: src/sedan_description/urdf/sedan.urdf.xacro (robot description, xacro)
@@ -226,5 +226,5 @@
        truth-vs-EKF yaw rate check run first to isolate real slip from
        estimator lag. -->
-    <xacro:macro name="wheel_friction" params="link slip:=0.01">
+    <xacro:macro name="wheel_friction" params="link slip:=0.00">
         <gazebo reference="${link}">
             <collision>
